File: E-Bike PCB.kicad_pcb (KiCad board)
At the start: 6 copper layers, 0 parts

Commit message: 1st PCB prototype traced
Parts:
- added BZ1: Buzzer, Buzzer_Beeper:MagneticBuzzer_PUI_AT-0927-TT-6-R, F.Cu at (-46.9, 109.2)
- added C11: 100nF, Capacitor_SMD:C_0603_1608Metric_Pad1.08x0.95mm_HandSolder, F.Cu at (-32.1, 108.2)
- added C12: 1nF, Capacitor_SMD:C_0603_1608Metric_Pad1.08x0.95mm_HandSolder, F.Cu at (-52.5, 117.7)
- added C13: 22µF, Capacitor_SMD:C_0805_2012Metric_Pad1.18x1.45mm_HandSolder, F.Cu at (-41.8, 117.9)
- added C14: 22µF, Capacitor_SMD:C_0805_2012Metric_Pad1.18x1.45mm_HandSolder, F.Cu at (-44.6, 117.9)
- added C15: 22µF, Capacitor_SMD:C_0805_2012Metric_Pad1.18x1.45mm_HandSolder, F.Cu at (-47.6, 117.9)
- added C16: 100nF, Capacitor_SMD:C_0603_1608Metric_Pad1.08x0.95mm_HandSolder, F.Cu at (-50.2, 117.7)
- added C17: 4.7µF, Capacitor_SMD:CP_Elec_6.3x7.7, F.Cu at (-27.4, 57.8)
- added C18: 100nF, Capacitor_SMD:C_0603_1608Metric_Pad1.08x0.95mm_HandSolder, F.Cu at (-29.2, 62.7)
- added C19: 1nF, Capacitor_SMD:C_0603_1608Metric_Pad1.08x0.95mm_HandSolder, F.Cu at (-29.2, 72.4)
- added C20: 4.7µF, Capacitor_SMD:CP_Elec_6.3x7.7, F.Cu at (-27.4, 77.2)
- added C21: 100nF, Capacitor_SMD:C_0603_1608Metric_Pad1.08x0.95mm_HandSolder, F.Cu at (-29.2, 82.2)
- added C27: 1nF, Capacitor_SMD:C_0603_1608Metric_Pad1.08x0.95mm_HandSolder, F.Cu at (-29.2, 64.4)
- added C28: 4.7µF, Capacitor_SMD:CP_Elec_6.3x7.7, F.Cu at (-27.4, 94.5)
- added D1: SMBJ5371B, Diode_SMD:D_SMB_Handsoldering, F.Cu at (-21.7, 39.0)
- added D10: LED, LED_SMD:LED_0603_1608Metric, F.Cu at (-90.1, 52.7)
- added D11: WS2812B, LED_SMD:LED_WS2812B_PLCC4_5.0x5.0mm_P3.2mm, F.Cu at (-59.0, 95.0)
- added D2: BZT52C3V3, Diode_SMD:D_SOD-123F, F.Cu at (-71.5, 74.2)
- added D3: BZT52B5V1S, Diode_SMD:D_SOD-323_HandSoldering, F.Cu at (-28.1, 101.1)
- added D4: LED, LED_SMD:LED_0603_1608Metric, F.Cu at (-90.1, 55.6)
- added D5: LED, LED_SMD:LED_0603_1608Metric, F.Cu at (-24.4, 114.7)
- added D6: LED, LED_SMD:LED_0603_1608Metric, F.Cu at (-90.1, 41.2)
- added D7: LED, LED_SMD:LED_0603_1608Metric, F.Cu at (-90.1, 44.1)
- added D8: LED, LED_SMD:LED_0603_1608Metric, F.Cu at (-90.1, 47.0)
- added D9: LED, LED_SMD:LED_0603_1608Metric, F.Cu at (-90.1, 49.8)
- added F1: 0154002.DRT, Fuse:Fuseholder_Littelfuse_Nano2_154x, F.Cu at (-30.1, 47.0)
- added FB2: FerriteBead, Inductor_SMD:L_1210_3225Metric, F.Cu at (-30.1, 68.2)
- added H1: MountingHole, MountingHole:MountingHole_3.2mm_M3_ISO7380, F.Cu at (-101.9, 30.5)
- added H2: MountingHole, MountingHole:MountingHole_3.2mm_M3_ISO7380, F.Cu at (-12.5, 30.5)
- added H3: MountingHole, MountingHole:MountingHole_3.2mm_M3_ISO7380, F.Cu at (-101.9, 123.5)
- added H4: MountingHole, MountingHole:MountingHole_3.2mm_M3_ISO7380, F.Cu at (-12.5, 123.5)
- added J1: 9-6437287-8, Legacy:TE_9-6437287-8, F.Cu at (-99.3, 97.0)
- added J11: Conn_01x02_Socket, Connector_Phoenix_MC_HighVoltage:PhoenixContact_MCV_1,5_2-G-5.08_1x02_P5.08mm_Vertical, F.Cu at (-40.2, 31.1)
- added J16: Conn_01x02_Socket, Connector_Phoenix_MC_HighVoltage:PhoenixContact_MCV_1,5_2-G-5.08_1x02_P5.08mm_Vertical, F.Cu at (-25.1, 31.1)
- added J2: Conn_01x07_Socket, Connector_PinSocket_2.54mm:PinSocket_1x07_P2.54mm_Vertical, F.Cu at (-13.1, 101.2)
- added J6: Conn_01x03_Socket, Connector_PinSocket_2.54mm:PinSocket_1x03_P2.54mm_Vertical, F.Cu at (-100.7, 66.9)
- added J7: Conn_01x04_Socket, Connector_PinSocket_2.54mm:PinSocket_1x04_P2.54mm_Vertical, F.Cu at (-64.9, 31.4)
- added J8: Conn_01x03_Socket, Connector_PinSocket_2.54mm:PinSocket_1x03_P2.54mm_Vertical, F.Cu at (-75.9, 31.4)
- added JP1: Jumper_2_Open, Jumper:SolderJumper-2_P1.3mm_Open_Pad1.0x1.5mm, F.Cu at (-73.3, 82.2)
- added JP10: SJ_BRG, Jumper:SolderJumper-2_P1.3mm_Bridged_Pad1.0x1.5mm, F.Cu at (-73.3, 85.3)
- added JP11: SJ_BRG, Jumper:SolderJumper-2_P1.3mm_Bridged_Pad1.0x1.5mm, F.Cu at (-38.1, 44.4)
- added JP2: SJ_BRG, Jumper:SolderJumper-2_P1.3mm_Bridged_Pad1.0x1.5mm, F.Cu at (-47.0, 80.4)
- added JP3: SJ_BRG, Jumper:SolderJumper-2_P1.3mm_Bridged_Pad1.0x1.5mm, F.Cu at (-72.8, 93.4)
- added JP4: SJ_BRG, Jumper:SolderJumper-2_P1.3mm_Bridged_Pad1.0x1.5mm, F.Cu at (-51.7, 91.7)
- added JP5: SJ_BRG, Jumper:SolderJumper-2_P1.3mm_Bridged_Pad1.0x1.5mm, F.Cu at (-76.3, 100.5)
- added JP6: SJ_BRG, Jumper:SolderJumper-2_P1.3mm_Bridged_Pad1.0x1.5mm, F.Cu at (-64.9, 103.4)
- added JP7: SLDJP_OPEN, Jumper:SolderJumper-2_P1.3mm_Open_RoundedPad1.0x1.5mm, F.Cu at (-67.4, 91.7)
- added JP8: SLDJP_OPEN, Jumper:SolderJumper-2_P1.3mm_Open_RoundedPad1.0x1.5mm, F.Cu at (-48.4, 91.7)
- added JP9: SJ_BRG, Jumper:SolderJumper-2_P1.3mm_Bridged_Pad1.0x1.5mm, F.Cu at (-72.2, 61.9)
- added L2: 16µH, Inductor_SMD:L_Coilcraft_XAL1060-XXX, F.Cu at (-34.8, 117.5)
- added L3: 10µH, Inductor_SMD:L_Changjiang_FXL0420, F.Cu at (-30.1, 87.0)
- added M1: ~, BRADES_Modules:RFID-RC522, B.Cu at (-59.0, 62.0)
- added Q2: CSD18534Q5A, Package_TO_SOT_SMD:TDSON-8-1, F.Cu at (-42.7, 44.3)
- added Q3: BSS123, Package_TO_SOT_SMD:SOT-23, F.Cu at (-68.6, 107.1)
- added Q4: BSS84, Package_TO_SOT_SMD:SOT-23, F.Cu at (-72.6, 104.7)
- added Q5: BSS123, Package_TO_SOT_SMD:SOT-23, F.Cu at (-76.2, 97.2)
- added Q6: BSS123, Package_TO_SOT_SMD:SOT-23, F.Cu at (-46.9, 100.0)
- added Q7: CSD18534Q5A, Package_TO_SOT_SMD:TDSON-8-1, F.Cu at (-20.2, 44.5)
- added Q8: BSS123, Package_TO_SOT_SMD:SOT-23, F.Cu at (-77.7, 81.5)
- added Q9: BSS123, Package_TO_SOT_SMD:SOT-23, F.Cu at (-71.4, 56.3)
- added R10: 100k, Resistor_SMD:R_0603_1608Metric_Pad0.98x0.95mm_HandSolder, F.Cu at (-28.0, 107.3)
- added R11: 820k, Resistor_SMD:R_0603_1608Metric_Pad0.98x0.95mm_HandSolder, F.Cu at (-28.0, 104.4)
- added R12: 64.9k, Resistor_SMD:R_0603_1608Metric_Pad0.98x0.95mm_HandSolder, F.Cu at (-37.9, 103.0)
- added R13: 115k, Resistor_SMD:R_0603_1608Metric_Pad0.98x0.95mm_HandSolder, F.Cu at (-34.7, 109.2)
- added R14: 28,7k, Resistor_SMD:R_0603_1608Metric_Pad0.98x0.95mm_HandSolder, F.Cu at (-36.5, 109.2)
- added R15: 100R, Resistor_SMD:R_0603_1608Metric_Pad0.98x0.95mm_HandSolder, F.Cu at (-43.5, 97.4)
- added R16: 100k, Resistor_SMD:R_0603_1608Metric_Pad0.98x0.95mm_HandSolder, F.Cu at (-46.9, 96.9)
- added R17: 100R, Resistor_SMD:R_0603_1608Metric_Pad0.98x0.95mm_HandSolder, F.Cu at (-38.6, 48.9)
- added R18: 100R, Resistor_SMD:R_0603_1608Metric_Pad0.98x0.95mm_HandSolder, F.Cu at (-72.0, 96.4)
- added R19: 100R, Resistor_SMD:R_0603_1608Metric_Pad0.98x0.95mm_HandSolder, F.Cu at (-72.5, 100.0)
- added R2: 100k, Resistor_SMD:R_0603_1608Metric_Pad0.98x0.95mm_HandSolder, F.Cu at (-41.5, 49.8)
- added R20: 100R, Resistor_SMD:R_0603_1608Metric_Pad0.98x0.95mm_HandSolder, F.Cu at (-64.2, 107.1)
- added R21: 1k, Resistor_SMD:R_0603_1608Metric_Pad0.98x0.95mm_HandSolder, F.Cu at (-50.0, 100.2)
- added R22: 100R, Resistor_SMD:R_0603_1608Metric_Pad0.98x0.95mm_HandSolder, F.Cu at (-78.6, 86.1)
- added R23: 100R, Resistor_SMD:R_0603_1608Metric_Pad0.98x0.95mm_HandSolder, F.Cu at (-68.3, 104.3)
- added R24: 100R, Resistor_SMD:R_0603_1608Metric_Pad0.98x0.95mm_HandSolder, F.Cu at (-71.3, 59.2)
- added R25: 100R, Resistor_SMD:R_0603_1608Metric_Pad0.98x0.95mm_HandSolder, F.Cu at (-28.0, 39.0)
- added R3: 100k, Resistor_SMD:R_0603_1608Metric_Pad0.98x0.95mm_HandSolder, F.Cu at (-65.7, 107.1)
- added R4: 100k, Resistor_SMD:R_0603_1608Metric_Pad0.98x0.95mm_HandSolder, F.Cu at (-72.0, 98.0)
- added R42: 330, Resistor_SMD:R_0603_1608Metric, F.Cu at (-86.1, 55.6)
- added R43: 330, Resistor_SMD:R_0603_1608Metric, F.Cu at (-26.1, 114.7)
- added R44: 330, Resistor_SMD:R_0603_1608Metric, F.Cu at (-86.1, 41.2)
- added R45: 330, Resistor_SMD:R_0603_1608Metric, F.Cu at (-86.1, 44.1)
- added R46: 330, Resistor_SMD:R_0603_1608Metric, F.Cu at (-86.1, 47.0)
- added R47: 330, Resistor_SMD:R_0603_1608Metric, F.Cu at (-86.1, 49.8)
- added R48: 330, Resistor_SMD:R_0603_1608Metric, F.Cu at (-86.1, 52.7)
- added R5: 100k, Resistor_SMD:R_0603_1608Metric_Pad0.98x0.95mm_HandSolder, F.Cu at (-76.8, 86.1)
- added R6: 180k, Resistor_SMD:R_0603_1608Metric_Pad0.98x0.95mm_HandSolder, F.Cu at (-74.9, 76.7)
- added R7: 100k, Resistor_SMD:R_0603_1608Metric_Pad0.98x0.95mm_HandSolder, F.Cu at (-68.1, 56.3)
- added R8: 10k, Resistor_SMD:R_0603_1608Metric_Pad0.98x0.95mm_HandSolder, F.Cu at (-74.9, 68.6)
- added R9: 100k, Resistor_SMD:R_0603_1608Metric_Pad0.98x0.95mm_HandSolder, F.Cu at (-72.6, 101.7)
- added TP1: TestPoint, TestPoint:TestPoint_Pad_1.5x1.5mm, F.Cu at (-24.9, 111.1)
- added TP3: TestPoint, TestPoint:TestPoint_Pad_1.5x1.5mm, F.Cu at (-74.9, 72.8)
- added TP4: TestPoint, TestPoint:TestPoint_Pad_1.5x1.5mm, F.Cu at (-72.5, 109.3)
- added U1: XIAO ESP32C6, Legacy:XIAO-ESP32C6-DIP, F.Cu at (-59.0, 77.8)
- added U2: LMR38020, Package_SO:Texas_HTSOP-8-1EP_3.9x4.9mm_P1.27mm_EP2.95x4.9mm_Mask2.4x3.1mm_ThermalVias, F.Cu at (-33.3, 103.0)
Routing:
- net LCD_LightSW: track 0.00 -> 151.9 mm, vias 0 -> 2
- net LCD_IGNITION: track 0.00 -> 142.6 mm
- net +5V: track 0.00 -> 140.8 mm, vias 0 -> 2
- net MZ_~{Brake_LOW}: track 0.00 -> 104.9 mm, vias 0 -> 1
- net LCD_TX: track 0.00 -> 99.4 mm
- net LCD_PWR+: track 0.00 -> 95.9 mm
- net LCD_GND: track 0.00 -> 95.7 mm
- net LCD_RX: track 0.00 -> 94.7 mm
- net GearSelect2: track 0.00 -> 78.9 mm, vias 0 -> 3
- net MZ_Throttle_Vdd: track 0.00 -> 66.3 mm, vias 0 -> 1
- net MZ_Throttle_Vcc: track 0.00 -> 65.8 mm, vias 0 -> 2
- net MZ_ThrottleSignal: track 0.00 -> 64.8 mm, vias 0 -> 1
- net GearSelect1: track 0.00 -> 61.8 mm, vias 0 -> 1
- net Throttle_Cutoff: track 0.00 -> 56.7 mm, vias 0 -> 1
- net MZ_Speed_Limit: track 0.00 -> 45.9 mm
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- added copper zone on B.Cu, net GND
- added copper zone on F.Cu, net GND
Other:
- board outline added: 96.4 x 100 mm
- board text added: "+5V"
- board text added: "BAT+"
- board text added: "BAT-"
- board text added: "BEAM"
- board text added: "BEAM+"
- board text added: "BEAM-"
- board text added: "BEAM_ON"
- board text added: "BRAKE"
- board text added: "BRK_FRONT"
- board text added: "BRK_GND"
- board text added: "BRK_REAR"
- board text added: "GEAR_SELECT1"
- board text added: "GEAR_SELECT2"
- board text added: "LCD"
- board text added: "LCD_GND"
- board text added: "LCD_IGNITION"
- board text added: "LCD_LIGHT_GND"
- board text added: "LCD_LightSW"
- board text added: "LCD_PWR+"
- board text added: "LCD_RX"
- board text added: "LCD_TX"
- board text added: "PAS"
- board text added: "PAS+"
- board text added: "PAS-"
- board text added: "PAS_SIG"
- board text added: "PWR_ENABLE"
- board text added: "SPD_LIM"
- board text added: "THR+"
- board text added: "THR-"
- board text added: "THROTTLE"
- board text added: "THR_CUT"
- board text added: "THR_SIG"
