File: Project Architecture.kicad_sch (KiCad schematic)
At the start: 0 parts

Commit message: 1st PCB prototype traced
Parts:
- added H1, H2, H3, H4: MountingHole, MountingHole:MountingHole_3.2mm_M3_ISO7380, symbol Mechanical:MountingHole
Other:
- sheet MCU renamed MCU (page 9)
