File: Section A - Title A.kicad_sch (KiCad schematic)
At the start: 1 part, among them U1 XIAO ESP32C6

Commit message: 1st PCB prototype traced
Parts:
- added JP4: SJ_BRG, Jumper:SolderJumper-2_P1.3mm_Bridged_Pad1.0x1.5mm, symbol Jumper:SolderJumper_2_Bridged
- added JP7, JP8: SLDJP_OPEN, Jumper:SolderJumper-2_P1.3mm_Open_RoundedPad1.0x1.5mm, symbol Jumper:SolderJumper_2_Open
- U1: footprint LEGACY:XIAO-ESP32C6-DIP -> Legacy:XIAO-ESP32C6-DIP
Connections:
- net ESP_WakeUp: now also U1.2 (D1); no longer U1.1 (D0)
- net GearSelect1: now also U1.4 (D3)
- net GearSelect2: now also U1.11 (D10)
- net MZ_RX: now also JP7.1 (A); no longer U1.7 (D6)
- net MZ_TX: now also JP8.2 (B); no longer U1.8 (D7)
- net BUZZER: now reaches U1.10 (D9)
- net +3.3V: now reaches U1.12 (VCC_3V3)
- net +5V: now reaches U1.14 (VUSB)
- net Throttle_Cutoff: now reaches U1.3 (D2)
- net SDA: now reaches U1.5 (D4)
- net SCL: now reaches U1.6 (D5)
- net MZ_~{Brake_LOW}: now reaches U1.9 (D8)
- new net: JP4.2 (B), JP8.1 (A), U1.8 (D7)
- new net: JP7.2 (B), U1.7 (D6)
- new net DEBUG_LED: JP4.1 (A)
- new net Speed_Limit: U1.1 (D0)
Other:
- note added: "According to the chip manual of ESP32C3, GPIO2, GPIO8 and GPIO9 in the chip are Strapping Pins, the high and low level configurations of these pins may allow the chip to enter into different Boot modes, please pay attention to this point when you use these pins, otherwise it may prevent your XIAO from uploading or executing the program all the time."
- note added: "Page 8"
- moved on the sheet: U1
