File: Section B - TItle B.kicad_sch (KiCad schematic)
At the start: 5 parts, among them Q1 CSD18534Q5A

Commit message: 1st PCB prototype traced
Parts:
- removed D1: BZT52C3V3, Diode_SMD:D_SOD-123F, symbol Device:D_Zener
- removed Q1: CSD18534Q5A, Package_TO_SOT_SMD:TDSON-8-1, symbol Transistor_FET:CSD18534Q5A
- removed R1: 100k, Resistor_SMD:R_0603_1608Metric_Pad0.98x0.95mm_HandSolder, symbol Device:R
- removed R5: 180k, Resistor_SMD:R_0603_1608Metric_Pad0.98x0.95mm_HandSolder, symbol Device:R
- removed R7: 10k, Resistor_SMD:R_0603_1608Metric_Pad0.98x0.95mm_HandSolder, symbol Device:R
Other:
- note removed: "1,91V - 2,87V"
- note removed: "36,4V - 54,6V"
