File: Section C - Title C.kicad_sch (KiCad schematic)
At the start: 6 parts, among them J11 Conn_01x02_Socket, J16 Conn_01x02_Socket, J2 Conn_01x07_Socket, J6 Conn_01x03_Socket, J7 Conn_01x04_Socket, J8 Conn_01x03_Socket

Commit message: 1st PCB prototype traced
Parts:
- added D1: SMBJ5371B, Diode_SMD:D_SMB_Handsoldering, symbol Device:D_Zener
- added Q7: CSD18534Q5A, Package_TO_SOT_SMD:TDSON-8-1, symbol Transistor_FET:CSD18534Q5A
- added R25: 100R, Resistor_SMD:R_0603_1608Metric_Pad0.98x0.95mm_HandSolder, symbol Device:R
- J11, J16: footprint (none) -> Connector_Phoenix_MC_HighVoltage:PhoenixContact_MCV_1,5_2-G-5.08_1x02_P5.08mm_Vertical
- J2: footprint (none) -> Connector_PinSocket_2.54mm:PinSocket_1x07_P2.54mm_Vertical
- J6, J8: footprint (none) -> Connector_PinSocket_2.54mm:PinSocket_1x03_P2.54mm_Vertical
- J7: footprint (none) -> Connector_PinSocket_2.54mm:PinSocket_1x04_P2.54mm_Vertical
Connections:
- net GND: now also D1.2 (A), Q7.1 (S), Q7.2 (S), Q7.3 (S); no longer J16.1 (Pin_1)
- net HighBeam_PWR+: now also J11.1 (Pin_1); no longer J11.2 (Pin_2)
- net HighBeam_PWR-: now also J11.2 (Pin_2); no longer J11.1 (Pin_1)
- net Vbat_{raw}: now also R25.1
- new net: J16.1 (Pin_1), Q7.5 (D)
- new net: D1.1 (K), Q7.4 (G), R25.2
Other:
- moved on the sheet: J11, J16
