File: Section E - Title E.kicad_sch (KiCad schematic)
At the start: 4 parts, among them J1 9-6437287-8, J10 Conn_01x04_Socket, J13 Conn_01x03_Socket, J9 Conn_01x03_Socket

Commit message: 1st PCB prototype traced
Parts:
- removed J10: Conn_01x04_Socket, symbol Connector:Conn_01x04_Socket
- removed J13, J9: Conn_01x03_Socket, symbol Connector:Conn_01x03_Socket
- J1: footprint LEGACY:TE_9-6437287-8 -> Legacy:TE_9-6437287-8
Connections:
- net LCD_GND: now also J1.14
- net LCD_IGNITION: now also J1.8
- net LCD_PWR+: now also J1.1
- net LCD_RX: now also J1.20
- net LCD_TX: now also J1.21
- net MZ_PasSignal: now also J1.6
- net MZ_Pas_Vcc: now also J1.7
- net MZ_Pas_Vdd: now also J1.13
- net MZ_ThrottleSignal: now also J1.26
- net MZ_Throttle_Vdd: now also J1.19
- net MZ_~{Brake_LOW}: now also J1.2
- net MZ_Throttle_Vcc-Provide: now reaches J1.25
- net MZ_3Speed: now reaches J1.3
- net MZ_Speed_Limit: now reaches J1.4
- no-connect marks 0 -> 12
Other:
- note added: "BLACK-WHITE"
- note added: "BLACK-YELLOW"
- note added: "GREEN-BLACK"
- note added: "Opis przewodów w sterowniku Sabvoton ML7260: Czarny [GND], Czerwony [+5V], Zielony [Hall], Niebieski [Hall], Żółty[ Hall] - złącze czujników Halla z silnika. Czerwono-Biały [+5V], czarny [GND], Zielony [sygnał] - manetka przyśpieszania manetki Szary [Duża prędkość], Czarny [GND], Niebieski [Mała prędkość] LUB Biało-Niebieski [Duża prędkość], Czarny [GND], Żółto-Biały [Mała prędkość] - Nastawy ogr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"
- note added: "RED-YELLOW"
- note removed: "REAR + FRONT Brake sensor"
- moved on the sheet: J1
