File: Section F - TItle F.kicad_sch (KiCad schematic)
At the start: 37 parts, among them U2 LMR38020

Commit message: 1st PCB prototype traced
Parts:
- added D3: BZT52B5V1S, Diode_SMD:D_SOD-323_HandSoldering, symbol Device:D_Zener
- added D5: LED, LED_SMD:LED_0603_1608Metric, symbol Device:LED
- added R43: 330, Resistor_SMD:R_0603_1608Metric, symbol Device:R
- added TP1: TestPoint, TestPoint:TestPoint_Pad_1.5x1.5mm, symbol Connector:TestPoint
- C1, C10, C2, C3, C4, C5, C6, C7, C9, FB1, L1: now not fitted; now left out of the parts list
- C11, C16, C18, C21: footprint (none) -> Capacitor_SMD:C_0603_1608Metric_Pad1.08x0.95mm_HandSolder; JLCPCB Part # (none) -> C15725; Manufacturer (none) -> CL10B104KC8NNNC
- C12, C19, C27: footprint (none) -> Capacitor_SMD:C_0603_1608Metric_Pad1.08x0.95mm_HandSolder; JLCPCB Part # (none) -> C77438; Manufacturer (none) -> 0603B102K101CT
- C13, C14, C15: footprint (none) -> Capacitor_SMD:C_0805_2012Metric_Pad1.18x1.45mm_HandSolder; JLCPCB Part # (none) -> C29277; Manufacturer (none) -> CL21A226MPQNNNE
- C17, C20, C28: footprint (none) -> Capacitor_SMD:CP_Elec_6.3x7.7; symbol Device:C -> Device:C_Polarized_US; JLCPCB Part # (none) -> C970653; Manufacturer (none) -> RVT2A4R7M0607 4.7UF 100V
- C8: symbol Device:C -> Device:C_Polarized_US; now not fitted; now left out of the parts list
- D4: JLCPCB Part # LTST-C190GKT -> C2286; Manufacturer (none) -> KT-0603R; now fitted; now in the parts list
- F1: Manufacturer (none) -> 0154002.DRT
- FB2: footprint Inductor_SMD:L_1206_3216Metric -> Inductor_SMD:L_1210_3225Metric; Manufacturer (none) -> CBG322513U601T
- L2: footprint Inductor_SMD:L_Changjiang_FXL0420 -> Inductor_SMD:L_Coilcraft_XAL1060-XXX
- R10: footprint (none) -> Resistor_SMD:R_0603_1608Metric_Pad0.98x0.95mm_HandSolder; JLCPCB Part # (none) -> C25803; Manufacturer (none) -> 0603WAF1003T5E
- R11: footprint (none) -> Resistor_SMD:R_0603_1608Metric_Pad0.98x0.95mm_HandSolder; JLCPCB Part # (none) -> C23252; Manufacturer (none) -> 0603WAF8203T5E
- R12: footprint (none) -> Resistor_SMD:R_0603_1608Metric_Pad0.98x0.95mm_HandSolder; JLCPCB Part # (none) -> C14891; Manufacturer (none) -> 0603WAF6492T5E
- R13: footprint (none) -> Resistor_SMD:R_0603_1608Metric_Pad0.98x0.95mm_HandSolder; JLCPCB Part # (none) -> C22783; Manufacturer (none) -> 0603WAF1153T5E
- R14: footprint (none) -> Resistor_SMD:R_0603_1608Metric_Pad0.98x0.95mm_HandSolder; JLCPCB Part # (none) -> C22928; Manufacturer (none) -> 0603WAF2872T5E
- R42: JLCPCB Part # CRCW0603330RFKEAHP -> C23138; Manufacturer (none) -> 0603WAF3300T5E; Vendor DigiKey -> (none); now fitted; now in the parts list
- U2: JLCPCB Part # (none) -> C3192337; Manufacturer (none) -> LMR38020SDDAR
Connections:
- net GND: now also D3.2 (A), D5.1 (K)
- net Vbat: now also U2.3 (VIN)
- net Vin: no longer U2.3 (VIN)
- net PWR_ENABLE: now reaches R10.2, R11.2, U2.2 (EN)
- net PWR_ENABLE: now also D3.1 (K), R43.2, TP1.1
- new net: D5.2 (A), R43.1
Other:
- moved on the sheet: R10, R11
